File: YAEWSBM2.kicad_sch (KiCad schematic)
At the start: 20 parts, among them J1 Conn_01x01_Pin, J2 Conn_01x01_Pin, J3 Conn_01x08_Pin, Q1 MMBT3904, Q2 MMBT3904

Commit message: silk art
Parts:
- J3: footprint Connector_PinHeader_2.54mm:PinHeader_1x08_P2.54mm_Horizontal -> Connector_PinHeader_2.54mm:PinHeader_1x08_P2.54mm_Vertical
Connections:
- net +12V: now also J3.6 (Pin_6); no longer J3.3 (Pin_3)
- net -12V: now also J3.5 (Pin_5); no longer J3.4 (Pin_4)
- net AMP_IN: now also J3.3 (Pin_3); no longer J3.6 (Pin_6)
- net AMP_OUT: now also J3.4 (Pin_4); no longer J3.5 (Pin_5)
- net AUDIO: now also J3.7 (Pin_7); no longer J3.2 (Pin_2)
- net AUX: now also J3.8 (Pin_8); no longer J3.1 (Pin_1)
- net GND: now also J3.1 (Pin_1); no longer J3.8 (Pin_8)
- net VCA_OUT: now also J3.2 (Pin_2); no longer J3.7 (Pin_7)
Other:
- moved on the sheet: J3
Changed lines of the file:
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@@
     )
   )
-  (symbol (lib_id "Connector:Conn_01x08_Pin") (at 180.848 99.06 180) (unit 1)
-    (in_bom yes) (on_board yes) (dnp no) (fields_autoplaced)
-    (property "Reference" "J3" (at 181.61 97.155 0)
+  (symbol (lib_id "Connector:Conn_01x08_Pin") (at 180.848 96.52 0) (mirror y) (unit 1)
+    (in_bom yes) (on_board yes) (dnp no)
+    (property "Reference" "J3" (at 181.61 98.425 0)
       (effects (font (size 1.27 1.27)) (justify right))
     )
-    (property "Value" "Conn_01x08_Pin" (at 181.61 99.695 0)
+    (property "Value" "Conn_01x08_Pin" (at 181.61 95.885 0)
       (effects (font (size 1.27 1.27)) (justify right))
     )
-    (property "Footprint" "Connector_PinHeader_2.54mm:PinHeader_1x08_P2.54mm_Horizontal" (at 180.848 99.06 0)
+    (property "Footprint" "Connector_PinHeader_2.54mm:PinHeader_1x08_P2.54mm_Vertical" (at 180.848 96.52 0)
       (effects (font (size 1.27 1.27)) hide)
     )
-    (property "Datasheet" "~" (at 180.848 99.06 0)
+    (property "Datasheet" "~" (at 180.848 96.52 0)
       (effects (font (size 1.27 1.27)) hide)
     )
